File: hardware/version102/tmc2209_devboard.kicad_sch (KiCad schematic)
At the start: 41 parts, among them J1 Conn_01x02_Male, J2 Conn_01x03_Pin, J4 motor_conn, J5 motor_conn, J6 motor_conn, SW1 SW_Push, U1 TMC2209-LA

Commit message: minor changed for version 1.3. Changed component number for JLC parts for R3 (was wrong) relates #3
Parts:
- R3: LCSC C17415 -> C340455
Changed lines of the file:
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@@
       (effects (font (size 1.27 1.27)) hide)
     )
-    (property "LCSC" "C17415" (at 100.838 199.136 0)
+    (property "LCSC" "C340455" (at 100.838 199.136 0)
       (effects (font (size 1.27 1.27)) hide)
     )
